File: Pro/PCB/Lily58_Pro.kicad_pcb (KiCad board)
At the start: 2 copper layers, 142.5 x 106.3 mm, 87 parts, among them J1 LED, J2 4PIN, J3 OLED, P1 i2c_pin, P2 i2c_pin, SW1 SW_PUSH, SW10 SW_PUSH, SW11 SW_PUSH, SW12 SW_PUSH, SW13 SW_PUSH, SW14 SW_PUSH, SW15 SW_PUSH, SW16 SW_PUSH, SW17 SW_PUSH, SW18 SW_PUSH, SW19 SW_PUSH, SW2 SW_PUSH, SW20 SW_PUSH, SW21 SW_PUSH, SW22 SW_PUSH, SW23 SW_PUSH, SW24 SW_PUSH, SW25 SW_PUSH, SW26 SW_PUSH, SW27 SW_PUSH, SW28 SW_PUSH, SW29 SW_PUSH, SW3 SW_PUSH, SW4 SW_PUSH, SW5 SW_PUSH, SW6 SW_PUSH, SW7 SW_PUSH, SW8 SW_PUSH, SW9 SW_PUSH, U1 ProMicro

Commit message: Add missing fooprints from the board
Parts:
- JP1, JP2, JP3, JP4, JP5, JP6, JP7, JP8: value (none) -> Jumper_NO_Small
Changed lines of the file:
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@@
-(kicad_pcb (version 20171130) (host pcbnew "(5.0.0-3-g5ebb6b6)")
+(kicad_pcb (version 20171130) (host pcbnew 5.1.4-e60b266~84~ubuntu19.04.1)
   (general
     (thickness 1.6)
@@
     (zone_45_only no)
     (trace_min 0.2)
-    (segment_width 0.2)
-    (edge_width 0.15)
     (via_size 0.4)
     (via_drill 0.3)
@@
     (uvia_min_size 0.2)
     (uvia_min_drill 0.1)
+    (edge_width 0.15)
+    (segment_width 0.2)
     (pcb_text_width 0.3)
     (pcb_text_size 1.5 1.5)
@@
       (effects (font (size 0.8128 0.8128) (thickness 0.1524)))
     )
-    (fp_text value "" (at -2.755 0 90) (layer F.SilkS) hide
+    (fp_text value Jumper_NO_Small (at -2.755 0 90) (layer F.SilkS) hide
       (effects (font (size 0.8128 0.8128) (thickness 0.15)))
     )
@@
       (effects (font (size 0.8128 0.8128) (thickness 0.1524)))
     )
-    (fp_text value "" (at -2.755 0 90) (layer F.SilkS) hide
+    (fp_text value Jumper_NO_Small (at -2.755 0 90) (layer F.SilkS) hide
       (effects (font (size 0.8128 0.8128) (thickness 0.15)))
     )
@@
       (effects (font (size 0.8128 0.8128) (thickness 0.1524)))
     )
-    (fp_text value "" (at -2.755 0 90) (layer F.SilkS) hide
+    (fp_text value Jumper_NO_Small (at -2.755 0 90) (layer F.SilkS) hide
       (effects (font (size 0.8128 0.8128) (thickness 0.15)))
     )
@@
       (effects (font (size 0.8128 0.8128) (thickness 0.1524)))
     )
-    (fp_text value "" (at -2.755 0 90) (layer F.SilkS) hide
+    (fp_text value Jumper_NO_Small (at -2.755 0 90) (layer F.SilkS) hide
       (effects (font (size 0.8128 0.8128) (thickness 0.15)))
     )
@@
       (effects (font (size 0.8128 0.8128) (thickness 0.1524)) (justify mirror))
     )
-    (fp_text value "" (at -2.755 0 90) (layer B.SilkS) hide
+    (fp_text value Jumper_NO_Small (at -2.755 0 90) (layer B.SilkS) hide
       (effects (font (size 0.8128 0.8128) (thickness 0.15)) (justify mirror))
     )
@@
       (effects (font (size 0.8128 0.8128) (thickness 0.1524)) (justify mirror))
     )
-    (fp_text value "" (at -2.755 0 90) (layer B.SilkS) hide
+    (fp_text value Jumper_NO_Small (at -2.755 0 90) (layer B.SilkS) hide
       (effects (font (size 0.8128 0.8128) (thickness 0.15)) (justify mirror))
     )
@@
       (effects (font (size 0.8128 0.8128) (thickness 0.1524)) (justify mirror))
     )
-    (fp_text value "" (at -2.755 0 90) (layer B.SilkS) hide
+    (fp_text value Jumper_NO_Small (at -2.755 0 90) (layer B.SilkS) hide
       (effects (font (size 0.8128 0.8128) (thickness 0.15)) (justify mirror))
     )
@@
       (effects (font (size 0.8128 0.8128) (thickness 0.1524)) (justify mirror))
     )
-    (fp_text value "" (at -2.755 0 90) (layer B.SilkS) hide
+    (fp_text value Jumper_NO_Small (at -2.755 0 90) (layer B.SilkS) hide
       (effects (font (size 0.8128 0.8128) (thickness 0.15)) (justify mirror))
     )
